File: Hardware/AT42QT1010_Capacitive_Touch_Breakout.sch (EAGLE design)
At the start: 20 parts, among them Q1 NPN

Commit message: started layout
Parts:
- added JP4: M01PTH, SparkFun-Connectors:M01PTH
- added JP7: NC, SparkFun-Passives:JUMPER-2SMD-NC
- added JP8: JUMPER-31-2, SparkFun-Passives:JUMPER-31-2
- JP1: value (none) -> M01PTH; device SparkFun-Connectors:M04PTH -> SparkFun-Connectors:M01PTH
- JP2: value (none) -> M01PTH; device SparkFun-Passives:JUMPER-2SMD-NC -> SparkFun-Connectors:M01PTH
- JP3: value JUMPER-31-2 -> M01PTH; device SparkFun-Passives:JUMPER-31-2 -> SparkFun-Connectors:M01PTH
Connections:
- removed net N$9: JP2.2, R2.1
- net GND: now also JP4.1, JP8.3; no longer JP1.3, JP3.3
- net LED: now also JP1.1, JP7.2, R2.1; no longer JP1.4
- net N$7: now also JP8.2; no longer JP3.2
- net OUT: now also JP3.1, JP7.1; no longer JP1.2, JP2.1
- net VCC: now also JP2.1, JP8.1; no longer JP1.1, JP3.1
Changed lines of the file:
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@@
 <setting verticaltext="up"/>
 </settings>
-<grid distance="0.1" unitdist="inch" unit="inch" style="lines" multiple="1" display="no" altdistance="0.01" altunitdist="inch" altunit="inch"/>
+<grid distance="0.1" unitdist="inch" unit="inch" style="lines" multiple="1" display="yes" altdistance="0.01" altunitdist="inch" altunit="inch"/>
 <layers>
 <layer number="1" name="Top" color="4" fill="1" visible="no" active="no"/>
@@
 <part name="SUPPLY2" library="SparkFun-Aesthetics" deviceset="VCC" device=""/>
 <part name="SUPPLY3" library="SparkFun-Aesthetics" deviceset="VCC" device=""/>
-<part name="JP1" library="SparkFun-Connectors" deviceset="M04" device="PTH"/>
 <part name="C1" library="SparkFun-Capacitors" deviceset="CAP" device="0603-CAP" value="0.1uF"/>
 <part name="C2" library="SparkFun-Capacitors" deviceset="CAP" device="0603-CAP" value="10nF"/>
@@
 <part name="Q1" library="SparkFun-DiscreteSemi" deviceset="TRANSISTOR_NPN" device="MMBT2222A" value="NPN"/>
 <part name="SUPPLY4" library="SparkFun-Aesthetics" deviceset="VCC" device=""/>
-<part name="JP2" library="SparkFun-Passives" deviceset="JUMPER-2" device="SMD-NC"/>
-<part name="JP3" library="SparkFun-Passives" deviceset="JUMPER-3" device="1-2"/>
+<part name="JP7" library="SparkFun-Passives" deviceset="JUMPER-2" device="SMD-NC" value="NC"/>
+<part name="JP8" library="SparkFun-Passives" deviceset="JUMPER-3" device="1-2"/>
 <part name="GND1" library="SparkFun-Aesthetics" deviceset="GND" device=""/>
 <part name="GND2" library="SparkFun-Aesthetics" deviceset="GND" device=""/>
@@
 <part name="LOGO1" library="SparkFun-Aesthetics" deviceset="LOGO-SFE" device="NEW"/>
 <part name="LOGO3" library="SparkFun-Aesthetics" deviceset="LOGO-SFE" device="SK"/>
+<part name="JP1" library="SparkFun-Connectors" deviceset="M01" device="PTH"/>
+<part name="JP2" library="SparkFun-Connectors" deviceset="M01" device="PTH"/>
+<part name="JP3" library="SparkFun-Connectors" deviceset="M01" device="PTH"/>
+<part name="JP4" library="SparkFun-Connectors" deviceset="M01" device="PTH"/>
 </parts>
 <sheets>
@@
 <instance part="LOGO2" gate="G$1" x="132.08" y="12.7"/>
 <instance part="SUPPLY1" gate="1" x="137.16" y="139.7"/>
-<instance part="SUPPLY2" gate="1" x="73.66" y="132.08"/>
+<instance part="SUPPLY2" gate="1" x="71.12" y="121.92"/>
 <instance part="SUPPLY3" gate="1" x="91.44" y="132.08"/>
-<instance part="JP1" gate="G$1" x="55.88" y="127" rot="MR180"/>
 <instance part="C1" gate="G$1" x="91.44" y="124.46"/>
 <instance part="C2" gate="G$1" x="165.1" y="127"/>
@@
 <instance part="Q1" gate="G$1" x="81.28" y="35.56"/>
 <instance part="SUPPLY4" gate="1" x="83.82" y="73.66"/>
-<instance part="JP2" gate="A" x="58.42" y="40.64"/>
-<instance part="JP3" gate="G$1" x="170.18" y="111.76" rot="R270"/>
-<instance part="GND1" gate="1" x="73.66" y="119.38"/>
+<instance part="JP7" gate="A" x="50.8" y="40.64"/>
+<instance part="JP8" gate="G$1" x="170.18" y="111.76" rot="R270"/>
+<instance part="GND1" gate="1" x="71.12" y="93.98"/>
 <instance part="GND2" gate="1" x="91.44" y="116.84"/>
 <instance part="GND3" gate="1" x="165.1" y="101.6"/>
@@
 <instance part="LOGO1" gate="G$1" x="241.3" y="25.4"/>
 <instance part="LOGO3" gate="G$1" x="231.14" y="25.4"/>
+<instance part="JP1" gate="G$1" x="50.8" y="129.54"/>
+<instance part="JP2" gate="G$1" x="50.8" y="119.38"/>
+<instance part="JP3" gate="G$1" x="50.8" y="109.22"/>
+<instance part="JP4" gate="G$1" x="50.8" y="99.06"/>
 </instances>
 <busses>
@@
 <net name="VCC" class="0">
 <segment>
-<pinref part="JP1" gate="G$1" pin="1"/>
-<pinref part="SUPPLY2" gate="1" pin="VCC"/>
-<wire x1="60.96" y1="129.54" x2="73.66" y2="129.54" width="0.1524" layer="91"/>
-<wire x1="73.66" y1="129.54" x2="73.66" y2="132.08" width="0.1524" layer="91"/>
-</segment>
-<segment>
 <pinref part="SUPPLY3" gate="1" pin="VCC"/>
 <pinref part="C1" gate="G$1" pin="1"/>
@@
 <pinref part="SUPPLY5" gate="1" pin="VCC"/>
 <wire x1="165.1" y1="114.3" x2="165.1" y2="111.76" width="0.1524" layer="91"/>
-<pinref part="JP3" gate="G$1" pin="1"/>
+<pinref part="JP8" gate="G$1" pin="1"/>
 <wire x1="165.1" y1="111.76" x2="167.64" y2="111.76" width="0.1524" layer="91"/>
 </segment>
@@
 <wire x1="137.16" y1="139.7" x2="137.16" y2="137.16" width="0.1524" layer="91"/>
 </segment>
+<segment>
+<pinref part="JP2" gate="G$1" pin="1"/>
+<pinref part="SUPPLY2" gate="1" pin="VCC"/>
+<wire x1="58.42" y1="119.38" x2="71.12" y2="119.38" width="0.1524" layer="91"/>
+<wire x1="71.12" y1="119.38" x2="71.12" y2="121.92" width="0.1524" layer="91"/>
+</segment>
 </net>
 <net name="GND" class="0">
-<segment>
-<pinref part="JP1" gate="G$1" pin="3"/>
-<pinref part="GND1" gate="1" pin="GND"/>
-<wire x1="60.96" y1="124.46" x2="73.66" y2="124.46" width="0.1524" layer="91"/>
-<wire x1="73.66" y1="124.46" x2="73.66" y2="121.92" width="0.1524" layer="91"/>
-</segment>
 <segment>
 <pinref part="C1" gate="G$1" pin="2"/>
@@
 </segment>
 <segment>
-<pinref part="JP3" gate="G$1" pin="3"/>
+<pinref part="JP8" gate="G$1" pin="3"/>
 <pinref part="GND3" gate="1" pin="GND"/>
 <wire x1="167.64" y1="106.68" x2="165.1" y2="106.68" width="0.1524" layer="91"/>
@@
 <wire x1="96.52" y1="33.02" x2="96.52" y2="27.94" width="0.1524" layer="91"/>
 </segment>
+<segment>
+<pinref part="JP4" gate="G$1" pin="1"/>
+<pinref part="GND1" gate="1" pin="GND"/>
+<wire x1="58.42" y1="99.06" x2="71.12" y2="99.06" width="0.1524" layer="91"/>
+<wire x1="71.12" y1="99.06" x2="71.12" y2="96.52" width="0.1524" layer="91"/>
+</segment>
 </net>
 <net name="OUT" class="0">
-<segment>
-<pinref part="JP1" gate="G$1" pin="2"/>
-<wire x1="60.96" y1="127" x2="68.58" y2="127" width="0.1524" layer="91"/>
-<label x="63.5" y="127" size="1.778" layer="95"/>
-</segment>
 <segment>
 <pinref part="U$1" gate="G$1" pin="OUT"/>
@@
 </segment>
 <segment>
-<pinref part="JP2" gate="A" pin="1"/>
-<wire x1="48.26" y1="35.56" x2="58.42" y2="35.56" width="0.1524" layer="91"/>
-<wire x1="58.42" y1="35.56" x2="58.42" y2="38.1" width="0.1524" layer="91"/>
-<label x="48.26" y="35.56" size="1.778" layer="95"/>
+<pinref part="JP7" gate="A" pin="1"/>
+<wire x1="40.64" y1="35.56" x2="50.8" y2="35.56" width="0.1524" layer="91"/>
+<wire x1="50.8" y1="35.56" x2="50.8" y2="38.1" width="0.1524" layer="91"/>
+<label x="40.64" y="35.56" size="1.778" layer="95"/>
+</segment>
+<segment>
+<pinref part="JP3" gate="G$1" pin="1"/>
+<wire x1="58.42" y1="109.22" x2="66.04" y2="109.22" width="0.1524" layer="91"/>
+<label x="60.96" y="109.22" size="1.778" layer="95"/>
 </segment>
 </net>
 <net name="LED" class="0">
 <segment>
-<pinref part="JP1" gate="G$1" pin="4"/>
-<wire x1="60.96" y1="121.92" x2="68.58" y2="121.92" width="0.1524" layer="91"/>
-<label x="63.5" y="121.92" size="1.778" layer="95"/>
+<pinref part="JP7" gate="A" pin="2"/>
+<wire x1="53.34" y1="38.1" x2="53.34" y2="35.56" width="0.1524" layer="91"/>
+<pinref part="R2" gate="G$1" pin="1"/>
+<wire x1="53.34" y1="35.56" x2="60.96" y2="35.56" width="0.1524" layer="91"/>
+<wire x1="60.96" y1="35.56" x2="66.04" y2="35.56" width="0.1524" layer="91"/>
+<wire x1="60.96" y1="48.26" x2="60.96" y2="35.56" width="0.1524" layer="91"/>
+<junction x="60.96" y="35.56"/>
+<label x="60.96" y="43.18" size="1.778" layer="95" rot="R90"/>
+</segment>
+<segment>
+<pinref part="JP1" gate="G$1" pin="1"/>
+<wire x1="58.42" y1="129.54" x2="66.04" y2="129.54" width="0.1524" layer="91"/>
+<label x="60.96" y="129.54" size="1.778" layer="95"/>
 </segment>
 </net>
@@
 <net name="N$7" class="0">
 <segment>
-<pinref part="JP3" gate="G$1" pin="2"/>
+<pinref part="JP8" gate="G$1" pin="2"/>
 <wire x1="167.64" y1="109.22" x2="157.48" y2="109.22" width="0.1524" layer="91"/>
 <wire x1="157.48" y1="109.22" x2="157.48" y2="116.84" width="0.1524" layer="91"/>
@@
 </segment>
 </net>
-<net name="N$9" class="0">
-<segment>
-<pinref part="JP2" gate="A" pin="2"/>
-<wire x1="60.96" y1="38.1" x2="60.96" y2="35.56" width="0.1524" layer="91"/>
-<pinref part="R2" gate="G$1" pin="1"/>
-<wire x1="60.96" y1="35.56" x2="66.04" y2="35.56" width="0.1524" layer="91"/>
-</segment>
-</net>

Commit message: Prototype board ready for review
Parts:
- added JP5: M01PTH, SparkFun-Connectors:M01PTH
- renumbered U$1 to U1, U$2 to D1
Connections:
- net PAD: now also JP5.1
Changed lines of the file:
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@@
 <?xml version="1.0" encoding="utf-8"?>
 <!DOCTYPE eagle SYSTEM "eagle.dtd">
-<eagle version="6.0">
+<eagle version="6.5.0">
 <drawing>
 <settings>
@@
 <setting verticaltext="up"/>
 </settings>
-<grid distance="0.1" unitdist="inch" unit="inch" style="lines" multiple="1" display="yes" altdistance="0.01" altunitdist="inch" altunit="inch"/>
+<grid distance="0.1" unitdist="inch" unit="inch" style="lines" multiple="1" display="no" altdistance="0.01" altunitdist="inch" altunit="inch"/>
 <layers>
 <layer number="1" name="Top" color="4" fill="1" visible="no" active="no"/>
+<layer number="2" name="Route2" color="1" fill="3" visible="no" active="no"/>
+<layer number="3" name="Route3" color="4" fill="3" visible="no" active="no"/>
+<layer number="4" name="Route4" color="1" fill="4" visible="no" active="no"/>
+<layer number="5" name="Route5" color="4" fill="4" visible="no" active="no"/>
+<layer number="6" name="Route6" color="1" fill="8" visible="no" active="no"/>
+<layer number="7" name="Route7" color="4" fill="8" visible="no" active="no"/>
+<layer number="8" name="Route8" color="1" fill="2" visible="no" active="no"/>
+<layer number="9" name="Route9" color="4" fill="2" visible="no" active="no"/>
+<layer number="10" name="Route10" color="1" fill="7" visible="no" active="no"/>
+<layer number="11" name="Route11" color="4" fill="7" visible="no" active="no"/>
+<layer number="12" name="Route12" color="1" fill="5" visible="no" active="no"/>
+<layer number="13" name="Route13" color="4" fill="5" visible="no" active="no"/>
+<layer number="14" name="Route14" color="1" fill="6" visible="no" active="no"/>
+<layer number="15" name="Route15" color="4" fill="6" visible="no" active="no"/>
 <layer number="16" name="Bottom" color="1" fill="1" visible="no" active="no"/>
 <layer number="17" name="Pads" color="2" fill="1" visible="no" active="no"/>
@@
 <classes>
 <class number="0" name="default" width="0" drill="0">
+<clearance class="0" value="0.205"/>
 </class>
 </classes>
 <parts>
-<part name="U$1" library="SparkFun-DigitalIC" deviceset="AT42QT1010" device="SOT23"/>
+<part name="U1" library="SparkFun-DigitalIC" deviceset="AT42QT1010" device="SOT23"/>
 <part name="FRAME1" library="SparkFun-Aesthetics" deviceset="FRAME-LETTER" device=""/>
 <part name="LOGO2" library="SparkFun-Aesthetics" deviceset="OSHW-LOGO" device="S"/>
@@
 <part name="R2" library="SparkFun-Resistors" deviceset="RESISTOR" device="0603" value="2.2k"/>
 <part name="R3" library="SparkFun-Resistors" deviceset="RESISTOR" device="0603" value="220"/>
-<part name="U$2" library="SparkFun-LED" deviceset="HSMC-C265" device=""/>
+<part name="D1" library="SparkFun-LED" deviceset="HSMC-C265" device=""/>
 <part name="Q1" library="SparkFun-DiscreteSemi" deviceset="TRANSISTOR_NPN" device="MMBT2222A" value="NPN"/>
 <part name="SUPPLY4" library="SparkFun-Aesthetics" deviceset="VCC" device=""/>
@@
 <part name="JP3" library="SparkFun-Connectors" deviceset="M01" device="PTH"/>
 <part name="JP4" library="SparkFun-Connectors" deviceset="M01" device="PTH"/>
+<part name="JP5" library="SparkFun-Connectors" deviceset="M01" device="PTH"/>
 </parts>
 <sheets>
@@
 </plain>
 <instances>
-<instance part="U$1" gate="G$1" x="137.16" y="121.92"/>
+<instance part="U1" gate="G$1" x="137.16" y="121.92"/>
 <instance part="FRAME1" gate="G$1" x="0" y="0"/>
 <instance part="FRAME1" gate="G$2" x="147.32" y="0"/>
@@
 <instance part="R2" gate="G$1" x="71.12" y="35.56"/>
 <instance part="R3" gate="G$1" x="83.82" y="66.04" rot="R90"/>
-<instance part="U$2" gate="G$1" x="83.82" y="50.8"/>
+<instance part="D1" gate="G$1" x="83.82" y="50.8"/>
 <instance part="Q1" gate="G$1" x="81.28" y="35.56"/>
 <instance part="SUPPLY4" gate="1" x="83.82" y="73.66"/>
@@
 <instance part="JP3" gate="G$1" x="50.8" y="109.22"/>
 <instance part="JP4" gate="G$1" x="50.8" y="99.06"/>
+<instance part="JP5" gate="G$1" x="198.12" y="124.46" rot="R180"/>
 </instances>
 <busses>
@@
 <segment>
 <pinref part="SUPPLY1" gate="1" pin="VCC"/>
-<pinref part="U$1" gate="G$1" pin="VDD"/>
+<pinref part="U1" gate="G$1" pin="VDD"/>
 <wire x1="137.16" y1="139.7" x2="137.16" y2="137.16" width="0.1524" layer="91"/>
 </segment>
@@
 </segment>
 <segment>
-<pinref part="U$1" gate="G$1" pin="VSS"/>
+<pinref part="U1" gate="G$1" pin="VSS"/>
 <pinref part="GND4" gate="1" pin="GND"/>
 <wire x1="119.38" y1="116.84" x2="116.84" y2="116.84" width="0.1524" layer="91"/>
@@
 <net name="OUT" class="0">
 <segment>
-<pinref part="U$1" gate="G$1" pin="OUT"/>
+<pinref part="U1" gate="G$1" pin="OUT"/>
 <wire x1="119.38" y1="127" x2="111.76" y2="127" width="0.1524" layer="91"/>
 <label x="111.76" y="127" size="1.778" layer="95"/>
@@
 <net name="N$4" class="0">
 <segment>
-<pinref part="U$1" gate="G$1" pin="SNS"/>
+<pinref part="U1" gate="G$1" pin="SNS"/>
 <pinref part="C2" gate="G$1" pin="2"/>
 <wire x1="154.94" y1="121.92" x2="165.1" y2="121.92" width="0.1524" layer="91"/>
@@
 <net name="N$5" class="0">
 <segment>
-<pinref part="U$1" gate="G$1" pin="SNSK"/>
+<pinref part="U1" gate="G$1" pin="SNSK"/>
 <wire x1="154.94" y1="127" x2="157.48" y2="127" width="0.1524" layer="91"/>
 <wire x1="157.48" y1="127" x2="157.48" y2="134.62" width="0.1524" layer="91"/>
@@
 <segment>
 <pinref part="R1" gate="G$1" pin="2"/>
-<wire x1="182.88" y1="134.62" x2="193.04" y2="134.62" width="0.1524" layer="91"/>
-<label x="187.96" y="134.62" size="1.778" layer="95"/>
+<wire x1="182.88" y1="134.62" x2="187.96" y2="134.62" width="0.1524" layer="91"/>
+<label x="195.58" y="134.62" size="1.778" layer="95"/>
+<pinref part="JP5" gate="G$1" pin="1"/>
+<wire x1="187.96" y1="134.62" x2="200.66" y2="134.62" width="0.1524" layer="91"/>
+<wire x1="190.5" y1="124.46" x2="187.96" y2="124.46" width="0.1524" layer="91"/>
+<wire x1="187.96" y1="124.46" x2="187.96" y2="134.62" width="0.1524" layer="91"/>
+<junction x="187.96" y="134.62"/>
 </segment>
 </net>
@@
 <wire x1="167.64" y1="109.22" x2="157.48" y2="109.22" width="0.1524" layer="91"/>
 <wire x1="157.48" y1="109.22" x2="157.48" y2="116.84" width="0.1524" layer="91"/>
-<pinref part="U$1" gate="G$1" pin="SYNC/MODE"/>
+<pinref part="U1" gate="G$1" pin="SYNC/MODE"/>
 <wire x1="157.48" y1="116.84" x2="154.94" y2="116.84" width="0.1524" layer="91"/>
 </segment>
@@
 <segment>
 <pinref part="Q1" gate="G$1" pin="C"/>
-<pinref part="U$2" gate="G$1" pin="C"/>
+<pinref part="D1" gate="G$1" pin="C"/>
 <wire x1="83.82" y1="40.64" x2="83.82" y2="43.18" width="0.1524" layer="91"/>
 <pinref part="C3" gate="G$1" pin="1"/>
@@
 <net name="N$12" class="0">
 <segment>
-<pinref part="U$2" gate="G$1" pin="A"/>
+<pinref part="D1" gate="G$1" pin="A"/>
 <pinref part="R3" gate="G$1" pin="1"/>
 <wire x1="83.82" y1="53.34" x2="83.82" y2="60.96" width="0.1524" layer="91"/>
